File: hardware/old/power.kicad_sch (KiCad schematic)
At the start: 36 parts, among them J1 MicroFit3.0_1x2, J2 XT60PW-M-AS, K1 CB1-P-12V, Q1 SI4946CDY-T1-GE3, Q2 IRF4905, U1 LTC4365TS8, U2 TMCS1100A2QDR, U3 R-78E5.0-1.0, U4 XL4015_Module

Commit message: Added power pcb sch + design
Parts:
- R79: value 10k -> 1.5k
- R88: value 1.5k -> 10k
Changed lines of the file:
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@@
 			)
 		)
-		(property "Value" "10k"
+		(property "Value" "1.5k"
 			(at 273.05 93.9799 0)
 			(effects
@@
 			)
 		)
-		(property "Value" "1.5k"
+		(property "Value" "10k"
 			(at 273.05 101.5999 0)
 			(effects
