File: hardware/logic-pcb/logic-pcb.kicad_sch (KiCad schematic)
At the start: 0 parts

Commit message: Add shunt for current measure
Parts:
- added C1, C4: 100n, symbol Device:C_Small
- added C2, C3, C5: 2200u, symbol Device:C_Polarized
- added J1, J2, J3: XT30, symbol Connector_Generic:Conn_01x02
- added R33: 10k, Resistor_SMD:R_0805_2012Metric_Pad1.20x1.40mm_HandSolder, symbol Device:R
- added U9: PCA9685PW, Package_SO:TSSOP-28_4.4x9.7mm_P0.65mm, symbol Driver_LED:PCA9685PW
Connections:
- new net: R33.1, U9.1 (A0), U9.2 (A1), U9.24 (A5), U9.3 (A2), U9.4 (A3), U9.5 (A4)
- new net +12V: C2.1, J3.2 (Pin_2)
- new net +3.3V: R33.2, U9.28 (VDD)
- new net +6V: C1.1, C3.1, C4.1, C5.1, J1.2 (Pin_2), J2.2 (Pin_2)
- new net ExtL.SIG_MB: U9.12 (LED6)
- new net ExtL.SIG_MM: U9.13 (LED7)
- new net ExtL.SIG_MS: U9.15 (LED8)
- new net ExtR.SIG_MB: U9.6 (LED0)
- new net ExtR.SIG_MM: U9.7 (LED1)
- new net ExtR.SIG_MS: U9.8 (LED2)
- new net GND: C1.2, C2.2, C3.2, C4.2, C5.2, J1.1 (Pin_1), J2.1 (Pin_1), J3.1 (Pin_1), U9.14 (VSS), U9.25 (EXTCLK)
- new net GRB_SIG_L: U9.20 (LED13)
- new net GRB_SIG_R: U9.19 (LED12)
- new net IntL.SIG_MB: U9.16 (LED9)
- new net IntL.SIG_MM: U9.17 (LED10)
- new net IntL.SIG_MS: U9.18 (LED11)
- new net IntR.SIG_MB: U9.9 (LED3)
- new net IntR.SIG_MM: U9.10 (LED4)
- new net IntR.SIG_MS: U9.11 (LED5)
- new net SCL: U9.26 (SCL)
- new net SDA: U9.27 (SDA)
- new net SIG_S_MAG: U9.21 (LED14)
- new net Servos_RST: U9.23 (~{OE})
- no-connect marks 0 -> 1
Other:
- note added: "Power IN"
- note added: "Servos PWM controRRer"
