File: hardware/logic-pcb/logic-pcb.kicad_sch (KiCad schematic)
At the start: 82 parts, among them J1 MicroFit2x2, J18 Conn_02x07_Odd_Even, J2 MicroFit2x2, J3 MicroFit2x12_Odd_Even, J5 MicroFit2x7, J6 XT30, SW1 RotaryEncoder_Switch, U1 NRF24L01_Breakout, U2 TCA9548APWR, U3 ESP32-S3-DevKitC, U4 TCA9555PWR, U6 R-78E3.3-1.0

Commit message: fixes pre-prod
Parts:
- removed R17, R21: 33R, Resistor_SMD:R_0805_2012Metric_Pad1.20x1.40mm_HandSolder, symbol Device:R_Small
- removed R27: 10k, Resistor_SMD:R_0805_2012Metric_Pad1.20x1.40mm_HandSolder, symbol Device:R
- added D1: 0805_Green, LED_SMD:LED_0805_2012Metric_Pad1.15x1.40mm_HandSolder, symbol Device:LED
- added R17: 1k, Resistor_SMD:R_0805_2012Metric_Pad1.20x1.40mm_HandSolder, symbol Device:R
- added R23: 10k, Resistor_SMD:R_0805_2012Metric_Pad1.20x1.40mm_HandSolder, symbol Device:R
- added R26, R27: 33R, Resistor_SMD:R_0805_2012Metric_Pad1.20x1.40mm_HandSolder, symbol Device:R_Small
- added TP1, TP2: TestPoint, TestPoint:TestPoint_THTPad_D1.0mm_Drill0.5mm, symbol Connector:TestPoint
- J18: symbol Connector_Generic:Conn_02x07_Odd_Even -> Connector_Generic:Conn_02x07_Top_Bottom; MPN 66201421122 -> 43045-1412; Manufacturer Wurth -> Molex
- J3: MPN 66202421122 -> 43045-2412; Manufacturer Wurth -> Molex
- J5: MPN 66201421122 -> 43045-1412; Manufacturer Wurth -> Molex
- J6: footprint Project:AMASS_XT30UPB-M_1x02_P5.0mm_Vertical -> Project:AMASS_XT30U-M_1x02_P5.0mm_Vertical
- R15: value 33R -> 10k; MPN CRCW080533R0FKEA -> CRCW080510K0FKEA
- R45: value 47k -> 10k; MPN CRCW080547K0FKEA -> CRCW080510K0FKEA
Connections:
- net +3V3: now also R15.2, TP1.1
- net +BATT: now also D1.2 (A)
- net BL.CS: now also J3.17 (Pin_17), R6.2; no longer J3.20 (Pin_20), R19.2
- net BL.D1: now also J3.18 (Pin_18); no longer J3.19 (Pin_19)
- net BL.DIR: now also J3.16 (Pin_16), R26.2; no longer J3.21 (Pin_21), R16.1
- net BL.STEP: now also J3.14 (Pin_14), R12.1; no longer J3.23 (Pin_23), R18.1
- net BR.CS: now also J3.5 (Pin_5), R27.2; no longer J3.8 (Pin_8), R14.2
- net BR.D1: now also J3.6 (Pin_6); no longer J3.7 (Pin_7)
- net BR.DIR: now also J3.4 (Pin_4), R22.2; no longer J3.9 (Pin_9), R10.1
- net BR.STEP: now also J3.2 (Pin_2), R10.1; no longer J3.11 (Pin_11), R12.1
- net FL.CS: now also J3.11 (Pin_11), R16.1; no longer J3.2 (Pin_2)
- net FL.D1: now also J3.12 (Pin_12); no longer J3.1 (Pin_1)
- net FL.DIR: now also J3.8 (Pin_8), R13.1; no longer J3.5 (Pin_5)
- net FL.STEP: now also J3.10 (Pin_10), R19.2; no longer J3.3 (Pin_3), R20.1
- net FR.CS: now also J3.23 (Pin_23), R14.2; no longer J3.14 (Pin_14), R15.2
- net FR.D1: now also J3.24 (Pin_24); no longer J3.13 (Pin_13)
- net FR.DIR: now also J3.20 (Pin_20); no longer J3.17 (Pin_17)
- net FR.STEP: now also J3.22 (Pin_22), R18.1; no longer J3.15 (Pin_15), R13.1
- net GND: now also J18.10 (Pin_10), J18.14 (Pin_14), J18.2 (Pin_2), J18.6 (Pin_6), J3.1 (Pin_1), J3.13 (Pin_13), J3.15 (Pin_15), J3.19 (Pin_19), J3.21 (Pin_21), J3.3 (Pin_3), J3.7 (Pin_7), J3.9 (Pin_9), R17.2, R23.2, TP2.1; no longer J18.1 (Pin_1), J18.13 (Pin_13), J18.5 (Pin_5), J18.9 (Pin_9), J3.10 (Pin_10), J3.12 (Pin_12), J3.16 (Pin_16), J3.18 (Pin_18), J3.22 (Pin_22), J3.24 (Pin_24), J3.4 (Pin_4), J3.6 (Pin_6)
- net LCD_CS: now also U3.7 (GPIO7/ADC1_CH6); no longer U3.16 (GPIO10/ADC1_CH9)
- net LCD_RS: now also U3.6 (GPIO6/ADC1_CH5), R23.1; no longer U3.17 (GPIO11/ADC2_CH0)
- net MISO: now also J18.9 (Pin_9), U3.17 (GPIO11/ADC2_CH0); no longer J18.11 (Pin_11), U3.27 (GPIO21)
- net MOSI: now also J18.13 (Pin_13), U3.27 (GPIO21); no longer J18.7 (Pin_7), R6.2
- net PROP_EN: now also J18.7 (Pin_7); no longer J18.2 (Pin_2)
- net SCK: now also J18.11 (Pin_11), R20.1; no longer J18.3 (Pin_3), R22.2
- net SCL_ACTUATION: now also J18.5 (Pin_5), U3.20 (GPIO14/ADC2_CH3); no longer J18.6 (Pin_6), U3.19 (GPIO13/ADC2_CH2)
- net SCL_SENSE: now also U3.5 (GPIO5/ADC1_CH4); no longer U3.10 (GPIO17/ADC2_CH6)
- net SDA_ACTUATION: now also J18.3 (Pin_3), U3.19 (GPIO13/ADC2_CH2); no longer J18.10 (Pin_10), U3.18 (GPIO12/ADC2_CH1)
- net SDA_SENSE: now also U3.4 (GPIO4/ADC1_CH3); no longer U3.20 (GPIO14/ADC2_CH3)
- net UOV_FAULT: now also J18.1 (Pin_1); no longer J18.14 (Pin_14)
- net ~{I2C_EXPANDER_RST}: now also U3.16 (GPIO10/ADC1_CH9); no longer U3.28 (GPIO47)
- net ~{IO_INT}: now also R15.1, U3.28 (GPIO47); no longer U3.15 (GPIO9/ADC1_CH8)
- net at R20.2: now also U3.18 (GPIO12/ADC2_CH1); no longer U3.6 (GPIO6/ADC1_CH5)
- new net: D1.1 (K), R17.1
- new net: R26.1, U3.10 (GPIO17/ADC2_CH6)
- new net: R27.1, U3.15 (GPIO9/ADC1_CH8)
Other:
- note added: "Monter ça un côté à l'endroit un côté l'envers comme ca c la mm"
- note added: "Power indicator"
- moved on the sheet: J18, R10, R11, R12, R13, R14, R16, R18, R19, R20, R22, R43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
