File: hardware/logic-pcb/logic-pcb.kicad_pcb (KiCad board)
At the start: 2 copper layers, 180 x 90 mm, 115 parts, among them J1 MicroFit2x2, J10 MicroFit2x2, J11 MicroFit2x2, J12 MicroFit2x2, J13 MicroFit2x2, J14 MicroFit2x2, J15 MicroFit2x2, J16 MicroFit2x2, J17 MicroFit2x2, J18 Conn_02x07_Odd_Even, J2 MicroFit2x2, J3 MicroFit2x12_Odd_Even, J5 MicroFit2x7, J6 XT30, J7 MicroFit2x2, J8 MicroFit2x2, J9 MicroFit2x2, SW1 RotaryEncoder_Switch, U1 NRF24L01_Breakout, U2 TCA9548APWR, U3 ESP32-S3-DevKitC, U4 TCA9555PWR, U6 R-78E3.3-1.0

Commit message: fixes pre-prod
Parts:
- removed R21: 33R, Resistor_SMD:R_0805_2012Metric_Pad1.20x1.40mm_HandSolder
- added D1: 0805_Green, LED_SMD:LED_0805_2012Metric_Pad1.15x1.40mm_HandSolder, F.Cu at (42.3, 69.1)
- added QR*****: Github QR, Project:Github QR, F.Cu at (37.4, 95.3)
- added R23: 10k, Resistor_SMD:R_0805_2012Metric_Pad1.20x1.40mm_HandSolder, B.Cu at (117.1, 68.9)
- added R26: 33R, Resistor_SMD:R_0805_2012Metric_Pad1.20x1.40mm_HandSolder, B.Cu at (164.3, 113.3)
- added TP1: TestPoint, TestPoint:TestPoint_THTPad_D1.0mm_Drill0.5mm, F.Cu at (80.5, 126.9)
- added TP2: TestPoint, TestPoint:TestPoint_THTPad_D1.0mm_Drill0.5mm, F.Cu at (72.2, 127.0)
- J6: footprint Project:AMASS_XT30UPB-M_1x02_P5.0mm_Vertical -> Project:AMASS_XT30U-M_1x02_P5.0mm_Vertical
- R1, R10, R12, R2, R20, R22, R24, R29, R31, R33, R35, R44, R6, R7, R8: moved to B.Cu
- R15: value 33R -> 10k; moved to B.Cu
- R17: value 33R -> 1k; moved to B.Cu
- R27: value 10k -> 33R; moved to B.Cu
- R45: value 47k -> 10k; moved to B.Cu
- moved R1 124.2 mm to (145.2, 119.4), turned to 180 degrees
- moved R2 122.3 mm to (149.6, 120.0), turned to -90 degrees
- moved R17 121.1 mm to (47.4, 69.1)
- moved R27 120.9 mm to (177.0, 113.2), turned to 90 degrees
- moved R10 116.4 mm to (159.2, 113.3), turned to -90 degrees
- moved R20 116.1 mm to (184.6, 113.2), turned to -90 degrees
- moved R7 112.8 mm to (187.4, 112.9), turned to 90 degrees
- moved R8 111.4 mm to (189.9, 112.9), turned to 90 degrees
- moved R12 111.1 mm to (161.8, 113.3), turned to -90 degrees
- moved R45 109.3 mm to (180.2, 119.3), turned to 180 degrees
- moved R6 108.7 mm to (169.4, 113.3), turned to 90 degrees
- moved R22 105.4 mm to (166.8, 113.3), turned to 90 degrees
- moved R15 94.7 mm to (182.2, 97.7), turned to -90 degrees
- moved C3 93.2 mm to (127.1, 125.8)
- moved R18 92.9 mm to (156.7, 90.6), turned to -90 degrees
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Connections:
- J18 pad 1: GND -> /UOV_FAULT
- J18 pad 10: /SDA_ACTUATION -> GND
- J18 pad 11: /MISO -> /SCK
- J18 pad 13: GND -> /MOSI
- J18 pad 14: /UOV_FAULT -> GND
- J18 pad 2: /PROP_EN -> GND
- J18 pad 3: /SCK -> /SDA_ACTUATION
- J18 pad 5: GND -> /SCL_ACTUATION
- J18 pad 6: /SCL_ACTUATION -> GND
- J18 pad 7: /MOSI -> /PROP_EN
- J18 pad 9: GND -> /MISO
- J3 pad 1: /FL.D1 -> GND
- J3 pad 10: GND -> /FL.STEP
- J3 pad 11: /BR.STEP -> /FL.CS
- J3 pad 12: GND -> /FL.D1
- J3 pad 13: /FR.D1 -> GND
- J3 pad 14: /FR.CS -> /BL.STEP
- J3 pad 15: /FR.STEP -> GND
- J3 pad 16: GND -> /BL.DIR
- J3 pad 17: /FR.DIR -> /BL.CS
- J3 pad 18: GND -> /BL.D1
- J3 pad 19: /BL.D1 -> GND
- J3 pad 2: /FL.CS -> /BR.STEP
- J3 pad 20: /BL.CS -> /FR.DIR
- J3 pad 21: /BL.DIR -> GND
- J3 pad 22: GND -> /FR.STEP
- J3 pad 23: /BL.STEP -> /FR.CS
- J3 pad 24: GND -> /FR.D1
- J3 pad 3: /FL.STEP -> GND
- J3 pad 4: GND -> /BR.DIR
- J3 pad 5: /FL.DIR -> /BR.CS
- J3 pad 6: GND -> /BR.D1
- J3 pad 7: /BR.D1 -> GND
- J3 pad 8: /BR.CS -> /FL.DIR
- J3 pad 9: /BR.DIR -> GND
- R10 pad 1: /BR.DIR -> /BR.STEP
- R12 pad 1: /BR.STEP -> /BL.STEP
- R13 pad 1: /FR.STEP -> /FL.DIR
- R14 pad 2: /BR.CS -> /FR.CS
- R15 pad 1: Net-(U3-GPIO4/ADC1_CH3) -> /~{IO_INT}
- R15 pad 2: /FR.CS -> +3V3
- R16 pad 1: /BL.DIR -> /FL.CS
- R17 pad 1: /FL.DIR -> Net-(D1-K)
- R17 pad 2: Net-(U3-GPIO5/ADC1_CH4) -> GND
- R18 pad 1: /BL.STEP -> /FR.STEP
- R19 pad 2: /BL.CS -> /FL.STEP
- R20 pad 1: /FL.STEP -> /SCK
- R20 pad 2: Net-(U3-GPIO6/ADC1_CH5) -> Net-(U3-GPIO12/ADC2_CH1)
- R22 pad 2: /SCK -> /BR.DIR
- R27 pad 1: /UOV_FAULT -> Net-(U3-GPIO9/ADC1_CH8)
- R27 pad 2: GND -> /BR.CS
- R6 pad 2: /MOSI -> /BL.CS
- U3 pad 10: /SCL_SENSE -> Net-(U3-GPIO17/ADC2_CH6)
- U3 pad 15: /~{IO_INT} -> Net-(U3-GPIO9/ADC1_CH8)
- U3 pad 16: /LCD_CS -> /~{I2C_EXPANDER_RST}
- U3 pad 17: /LCD_RS -> /MISO
- U3 pad 18: /SDA_ACTUATION -> Net-(U3-GPIO12/ADC2_CH1)
- U3 pad 19: /SCL_ACTUATION -> /SDA_ACTUATION
- U3 pad 20: /SDA_SENSE -> /SCL_ACTUATION
- U3 pad 27: /MISO -> /MOSI
- U3 pad 28: /~{I2C_EXPANDER_RST} -> /~{IO_INT}
- U3 pad 4: Net-(U3-GPIO4/ADC1_CH3) -> /SDA_SENSE
- U3 pad 5: Net-(U3-GPIO5/ADC1_CH4) -> /SCL_SENSE
- U3 pad 6: Net-(U3-GPIO6/ADC1_CH5) -> /LCD_RS
- U3 pad 7: Net-(U3-GPIO7/ADC1_CH6) -> /LCD_CS
Routing:
- net +3V3: track 443.1 -> 656.2 mm, vias 5 -> 14
- net /SCK: track 0.00 -> 206.7 mm, vias 0 -> 2
- net /MISO: track 0.00 -> 199.8 mm, vias 0 -> 1
- net /MOSI: track 0.00 -> 199.5 mm, vias 0 -> 3
- net /SCL_ACTUATION: track 0.00 -> 193.5 mm, vias 0 -> 4
- net /SCL_SENSE: track 0.00 -> 192.5 mm, vias 0 -> 3
- net /SDA_ACTUATION: track 0.00 -> 189.1 mm, vias 0 -> 5
- net /SDA_SENSE: track 0.00 -> 177.8 mm, vias 0 -> 3
- net Net-(U4-P07): track 0.00 -> 83.1 mm, vias 0 -> 1
- net /BR.CS: track 0.00 -> 82.2 mm
- net /UOV_FAULT: track 0.00 -> 78.1 mm, vias 0 -> 1
- net /LCD_RS: track 0.00 -> 73.3 mm, vias 0 -> 2
- net /BR.DIR: track 0.00 -> 72.0 mm
- net /BL.CS: track 0.00 -> 71.4 mm
- net /LCD_CS: track 0.00 -> 70.0 mm, vias 0 -> 2
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Other:
- board size 180 x 90 mm -> 175 x 90 mm
- board text added: "+3V3"
- board text added: "6V-16.8V ~0.5-1A"
- board text added: "BATT"
- board text added: "E.L."
- board text added: "E.R."
- board text added: "GND"
- board text added: "Game Team"
- board text added: "I.L."
- board text added: "I.R."
- board text added: "I2C - OUTPUTS"
- board text added: "I2C ACT."
- board text added: "I2C SENSE"
- board text added: "In Robots, We Trust"
- board text added: "LOGIC PCB"
- board text added: "Misc. Data"
- board text added: "Motors"
- board text added: "POWER LINK"
- board text added: "Rev ${REVISION}"
- board text added: "SCREEN"
- board text added: "TEST POINTS"
- board text added: "VL53L0X - BACK"
- board text added: "VL53L0X - FRONT"
