File: hardware/kinetic-pcb/kinetic-pcb.kicad_pcb (KiCad board)
At the start: 2 copper layers, 200 x 120 mm, 231 parts, among them J1 XT30, J10 MicroFit2x2, J11 MicroFit2x2, J12 MicroFit2x2, J13 MicroFit2x2, J14 MicroFit2x2, J15 MicroFit2x1, J16 MicroFit2x7, J17 MicroFit2x2, J18 MicroFit2x2, J19 MicroFit2x2, J2 XT30, J20 MicroFit2x2, J21 MicroFit2x7, J22 MicroFit2x7, J23 MicroFit2x1, J24 MicroFit2x1, J25 MicroFit2x1, J26 MicroFit2x1, J27 MicroFit2x1, J28 MicroFit2x1, J29 MicroFit2x7, J3 MicroFit2x2, J30 MicroFit2x7, J31 MicroFit2x7, J32 MicroFit2x7, J33 MicroFit2x1, J34 MicroFit2x7, J35 MicroFit2x2, J36 MicroFit2x2, J4 MicroFit2x2, J5 MicroFit2x2, J6 MicroFit2x2, J7 MicroFit2x2, J8 MicroFit2x2, J9 MicroFit2x2, Q1 DMN2053UQ-13, Q10 DMN2053UQ-13, Q11 DMN2053UQ-13, Q12 DMN2053UQ-13, Q2 DMN2053UQ-13, Q3 DMN2053UQ-13, Q4 DMN2053UQ-13, Q5 DMN2053UQ-13, Q6 DMN2053UQ-13, Q7 DMN2053UQ-13, Q8 DMN2053UQ-13, Q9 DMN2053UQ-13, U1 PCA9685PW, U2 TCA9555PWR, U3 R-78E3.3-1.0, U4 TCA9548APWR, U5 PCA9685PW, U6 PCA9685PW, U7 ISO1540, U8 ISO1540

Commit message: fixes pre-prod
Parts:
- removed R48, R50, R53, R55: 1k, Resistor_SMD:R_0805_2012Metric_Pad1.20x1.40mm_HandSolder
- added D12: 0805_Green, LED_SMD:LED_0805_2012Metric_Pad1.15x1.40mm_HandSolder, F.Cu at (78.8, 29.4)
- added R61: 1k, Resistor_SMD:R_0805_2012Metric_Pad1.20x1.40mm_HandSolder, B.Cu at (113.8, 48.4)
- J1, J2: footprint Project:AMASS_XT30UPB-M_1x02_P5.0mm_Vertical -> Project:AMASS_XT30U-M_1x02_P5.0mm_Vertical
- Q1, Q10, Q11, Q12, Q2, Q3, Q4, Q5, Q6, Q7, Q8, Q9: footprint Package_TO_SOT_SMD:TSOT-23_HandSoldering -> Project:SOT-23_Handsoldering-DMN2053UQ
- R47, R49, R54, R56: value 1k -> 4.7k
- moved R37 5.59 mm to (212.5, 117.5)
- moved R39 5.59 mm to (228.7, 130.1)
- moved R43 5.58 mm to (212.3, 130.2)
- moved R41 5.58 mm to (228.6, 118.3)
- moved R38 5.35 mm to (212.6, 112.0)
- moved R44 5.35 mm to (212.4, 124.7)
- moved R42 5.35 mm to (228.7, 112.8)
- moved R40 5.35 mm to (228.8, 124.6)
- moved Q6 2.11 mm to (227.9, 127.3), turned to 180 degrees
- moved Q7 2.11 mm to (227.8, 115.5), turned to 180 degrees
- moved Q8 2.11 mm to (211.5, 127.4), turned to 180 degrees
- moved Q5 2.11 mm to (211.7, 114.7), turned to 180 degrees
- moved Q2 2.11 mm to (84.0, 114.5), turned to 0 degrees
- moved Q3 2.11 mm to (84.2, 127.3), turned to 0 degrees
- moved Q4 2.11 mm to (67.3, 114.9), turned to 0 degrees
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Connections:
- C1 pad 1: GND -> +3V3
- C1 pad 2: +3V3 -> GND
- C11 pad 1: GND -> +3V3
- C11 pad 2: +3V3 -> GND
- C15 pad 1: GND -> +3V3
- C15 pad 2: +3V3 -> GND
- C21 pad 1: GND -> +3V3
- C21 pad 2: +3V3 -> GND
- C3 pad 1: GND -> +3V3
- C3 pad 2: +3V3 -> GND
- C59 pad 1: /I2C Sporadic/3V3D -> /I2C Sporadic/GNDD
- C59 pad 2: /I2C Sporadic/GNDD -> /I2C Sporadic/3V3D
- C63 pad 1: /I2C Realtime/3V3D -> /I2C Realtime/GNDD
- C63 pad 2: /I2C Realtime/GNDD -> /I2C Realtime/3V3D
- J10 pad 3: unconnected-(J10-Pin_3-Pad3) -> GND
- J10 pad 4: GND -> unconnected-(J10-Pin_4-Pad4)
- J11 pad 2: GND -> /Left Side/GRB_FRONT
- J11 pad 3: /Left Side/GRB_FRONT -> GND
- J12 pad 2: GND -> /Left Side/GRB_BACK
- J12 pad 3: unconnected-(J12-Pin_3-Pad3) -> GND
- J12 pad 4: /Left Side/GRB_BACK -> unconnected-(J12-Pin_4-Pad4)
- J13 pad 2: GND -> /Left Side/TURNER
- J13 pad 3: unconnected-(J13-Pin_3-Pad3) -> GND
- J13 pad 4: /Left Side/TURNER -> unconnected-(J13-Pin_4-Pad4)
- J14 pad 2: GND -> /Left Side/TURNER_HOLDER
- J14 pad 3: unconnected-(J14-Pin_3-Pad3) -> GND
- J14 pad 4: /Left Side/TURNER_HOLDER -> unconnected-(J14-Pin_4-Pad4)
- J17 pad 2: GND -> /Right Side/GRB_FRONT
- J17 pad 3: /Right Side/GRB_FRONT -> GND
- J18 pad 2: GND -> /Right Side/GRB_BACK
- J18 pad 3: unconnected-(J18-Pin_3-Pad3) -> GND
- J18 pad 4: /Right Side/GRB_BACK -> unconnected-(J18-Pin_4-Pad4)
- J19 pad 2: GND -> /Right Side/TURNER
- J19 pad 3: unconnected-(J19-Pin_3-Pad3) -> GND
- J19 pad 4: /Right Side/TURNER -> unconnected-(J19-Pin_4-Pad4)
- J20 pad 2: GND -> /Right Side/TURNER_HOLDER
- J20 pad 3: unconnected-(J20-Pin_3-Pad3) -> GND
- J20 pad 4: /Right Side/TURNER_HOLDER -> unconnected-(J20-Pin_4-Pad4)
- J6 pad 1: /STOCK_ISLAND -> +6V
- J6 pad 2: +6V -> /STOCK_ISLAND
- J6 pad 3: unconnected-(J6-Pin_3-Pad3) -> GND
- J6 pad 4: GND -> unconnected-(J6-Pin_4-Pad4)
- J7 pad 3: unconnected-(J7-Pin_3-Pad3) -> GND
- J7 pad 4: GND -> unconnected-(J7-Pin_4-Pad4)
- J8 pad 3: unconnected-(J8-Pin_3-Pad3) -> GND
- J8 pad 4: GND -> unconnected-(J8-Pin_4-Pad4)
- J9 pad 3: unconnected-(J9-Pin_3-Pad3) -> GND
- J9 pad 4: GND -> unconnected-(J9-Pin_4-Pad4)
- R47 pad 1: +3V3 -> SDA_SPORADIC
- R47 pad 2: Net-(R47-Pad2) -> +3V3
- R49 pad 1: Net-(R49-Pad1) -> +3V3
- R54 pad 1: Net-(R53-Pad2) -> SDA_REALTIME
- R54 pad 2: SDA_REALTIME -> +3V3
- R56 pad 2: Net-(R55-Pad1) -> SCL_REALTIME
Routing:
- net +12V: track 493.9 -> 603.8 mm, vias 1 -> 4
- net Net-(D12-K): track 0.00 -> 41.3 mm, vias 0 -> 1
- net GND: track 87.4 -> 119.8 mm, vias 944 -> 956
- net /FRONT_EXT_R_P: track 78.2 -> 83.8 mm
- net /BACK_EXT_R_P: track 80.7 -> 86.3 mm
- net /FRONT_INT_R_P: track 62.2 -> 67.7 mm
- net /Left Side/GRB_FRONT: track 51.4 -> 47.2 mm
- net /Right Side/GRB_BACK: track 68.8 -> 72.4 mm
- net /Left Side/TURNER_HOLDER: track 34.4 -> 31.4 mm
- net /Right Side/TURNER_HOLDER: track 30.6 -> 27.6 mm
- net Net-(D10-A): track 10.6 -> 13.5 mm
- net /Led Red/OUT: track 20.7 -> 23.6 mm
- net /Led Blue/OUT: track 30.4 -> 33.2 mm
- net Net-(D8-A): track 10.5 -> 13.3 mm
- net Net-(D9-A): track 10.6 -> 13.4 mm
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Other:
- outline, holes or cut-outs redrawn
- board text added: "+"
- board text added: "-"
- board text added: "I2C - Actuation"
- board text added: "I2C - Sense"
- board text added: "Rev ${REVISION}"
- board text removed: "I2C - Realtime"
- board text removed: "I2C - Sporadic"
- board text removed: "v${REVISION}"
