File: hardware/kinetic-pcb/kinetic-pcb.kicad_sch (KiCad schematic)
At the start: 70 parts, among them J1 XT30, J10 MicroFit2x2, J2 XT30, J3 MicroFit2x2, J4 MicroFit2x2, J5 MicroFit2x2, J6 MicroFit2x2, J7 MicroFit2x2, J8 MicroFit2x2, J9 MicroFit2x2, Q1 DMN2053UQ-13, U1 PCA9685PW, U2 TCA9555PWR, U3 R-78E3.3-1.0, U4 TCA9548APWR

Commit message: Adapt Power PCB to logic requirements
Parts:
- D1, D2: MPN (none) -> SS10P4-M3/87A; Manufacturer (none) -> Vishay
Other:
- company: (none) -> Game Team SLSC
- title: (none) -> Kinetic PCB
Changed lines of the file:
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@@
 	(generator_version "9.0")
 	(paper "A3")
+	(title_block
+		(title "Kinetic PCB")
+		(date "2026-03-12")
+		(rev "${REVISION}")
+		(company "Game Team SLSC")
+	)
 	(bus_alias "ArmPWM"
 		(members "SB" "SE" "SV")
@@
 			)
 		)
+		(property "MPN" "SS10P4-M3/87A "
+			(at 35.56 31.75 90)
+			(effects
+				(font
+					(size 1.27 1.27)
+				)
+				(hide yes)
+			)
+		)
+		(property "Manufacturer" "Vishay"
+			(at 35.56 31.75 90)
+			(effects
+				(font
+					(size 1.27 1.27)
+				)
+				(hide yes)
+			)
+		)
 		(pin "2"
 		)
@@
 			)
 		)
+		(property "MPN" "SS10P4-M3/87A "
+			(at 36.83 54.61 90)
+			(effects
+				(font
+					(size 1.27 1.27)
+				)
+				(hide yes)
+			)
+		)
+		(property "Manufacturer" "Vishay"
+			(at 36.83 54.61 90)
+			(effects
+				(font
+					(size 1.27 1.27)
+				)
+				(hide yes)
+			)
+		)
 		(pin "2"
 		)
@@
 		)
 		(instances
-			(project "logic-pcb"
+			(project "kinetic-pcb"
 				(path "/27daf012-9196-46de-9851-628d059dd653"
 					(page "32")
@@
 		)
 		(instances
-			(project "logic-pcb"
+			(project "kinetic-pcb"
 				(path "/27daf012-9196-46de-9851-628d059dd653"
 					(page "33")
@@
 		)
 		(instances
-			(project "logic-pcb"
+			(project "kinetic-pcb"
 				(path "/27daf012-9196-46de-9851-628d059dd653"
 					(page "2")
@@
 		)
 		(instances
-			(project "logic-pcb"
+			(project "kinetic-pcb"
 				(path "/27daf012-9196-46de-9851-628d059dd653"
 					(page "34")
@@
 		)
 		(instances
-			(project "logic-pcb"
+			(project "kinetic-pcb"
 				(path "/27daf012-9196-46de-9851-628d059dd653"
 					(page "35")
@@
 		)
 		(instances
-			(project "logic-pcb"
+			(project "kinetic-pcb"
 				(path "/27daf012-9196-46de-9851-628d059dd653"
 					(page "36")
@@
 		)
 		(instances
-			(project "logic-pcb"
+			(project "kinetic-pcb"
 				(path "/27daf012-9196-46de-9851-628d059dd653"
 					(page "23")
@@
 		)
 		(instances
-			(project "logic-pcb"
+			(project "kinetic-pcb"
 				(path "/27daf012-9196-46de-9851-628d059dd653"
 					(page "6")

Commit message: fixes pre-prod
Parts:
- removed C1, C11, C3: 10u, Capacitor_SMD:C_0805_2012Metric_Pad1.18x1.45mm_HandSolder, symbol Device:C_Polarized_Small
- added C1, C11, C3: 10u, Capacitor_SMD:C_0805_2012Metric_Pad1.18x1.45mm_HandSolder, symbol Device:C_Small
- added D12: 0805_Green, LED_SMD:LED_0805_2012Metric_Pad1.15x1.40mm_HandSolder, symbol Device:LED
- added R61: 1k, Resistor_SMD:R_0805_2012Metric_Pad1.20x1.40mm_HandSolder, symbol Device:R
- J1, J2: footprint Project:AMASS_XT30UPB-M_1x02_P5.0mm_Vertical -> Project:AMASS_XT30U-M_1x02_P5.0mm_Vertical
- J10, J6, J7, J8, J9: symbol Connector_Generic:Conn_02x02_Counter_Clockwise -> Connector_Generic:Conn_02x02_Top_Bottom
- Q1: footprint Package_TO_SOT_SMD:TSOT-23_HandSoldering -> Project:SOT-23_Handsoldering-DMN2053UQ
Connections:
- net +12V: now also D12.2 (A)
- net +3V3: now also C1.1, C11.1, C3.1
- net GND: now also J10.3 (Pin_3), J6.3 (Pin_3), J7.3 (Pin_3), J8.3 (Pin_3), J9.3 (Pin_3), C1.2, C11.2, C3.2, R61.2; no longer J10.4 (Pin_4), J6.4 (Pin_4), J7.4 (Pin_4), J8.4 (Pin_4), J9.4 (Pin_4)
- net STOCKMISC_PWR: now also J6.1 (Pin_1); no longer J6.2 (Pin_2)
- net STOCK_ISLAND: now also J6.2 (Pin_2); no longer J6.1 (Pin_1)
- new net: D12.1 (K), R61.1
Other:
- note added: "Power indicator"
- moved on the sheet: C12, H1, H2, H3, H4, J3, J4, R11, R14, R15, R16, U4
