File: hardware/kinetic-pcb/sheets/action-side.kicad_sch (KiCad schematic)
At the start: 20 parts, among them J11 MicroFit2x2, J12 MicroFit2x2, J13 MicroFit2x2, J14 MicroFit2x2, U5 PCA9685PW

Commit message: fixes pre-prod
Parts:
- removed C15: 10u, Capacitor_SMD:C_0805_2012Metric_Pad1.18x1.45mm_HandSolder, symbol Device:C_Polarized_Small
- added C15: 10u, Capacitor_SMD:C_0805_2012Metric_Pad1.18x1.45mm_HandSolder, symbol Device:C_Small
- J11, J12, J13, J14: symbol Connector_Generic:Conn_02x02_Odd_Even -> Connector_Generic:Conn_02x02_Top_Bottom
Connections:
- net +3V3: now also C15.1
- net GND: now also J11.3 (Pin_3), J12.3 (Pin_3), J13.3 (Pin_3), J14.3 (Pin_3), C15.2; no longer J11.2 (Pin_2), J12.2 (Pin_2), J13.2 (Pin_2), J14.2 (Pin_2)
- net GRB_BACK: now also J12.2 (Pin_2); no longer J12.4 (Pin_4)
- net GRB_FRONT: now also J11.2 (Pin_2); no longer J11.3 (Pin_3)
- net TURNER: now also J13.2 (Pin_2); no longer J13.4 (Pin_4)
- net TURNER_HOLDER: now also J14.2 (Pin_2); no longer J14.4 (Pin_4)
Other:
- moved on the sheet: J13, J14
