File: hardware/kinetic-pcb/sheets/arm.kicad_sch (KiCad schematic)
At the start: 1 part, among them J16 MicroFit2x7

Commit message: fixes pre-prod
Parts:
- J16: MPN 66201421122 -> 43045-1412; Manufacturer Wurth -> Molex
Changed lines of the file:
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@@
 			)
 		)
-		(property "MPN" "66201421122"
+		(property "MPN" "43045-1412"
 			(at 130.81 69.85 0)
 			(effects
@@
 			)
 		)
-		(property "Manufacturer" "Wurth"
+		(property "Manufacturer" "Molex"
 			(at 130.81 69.85 0)
 			(effects
