File: hardware/kinetic-pcb/sheets/i2c-source.kicad_sch (KiCad schematic)
At the start: 10 parts, among them J35 MicroFit2x2, U7 ISO1540

Commit message: fixes pre-prod
Parts:
- removed C59, C60: 10u, Capacitor_SMD:C_0805_2012Metric_Pad1.18x1.45mm_HandSolder, symbol Device:C_Polarized_Small
- removed R47, R48, R49, R50: 1k, Resistor_SMD:R_0805_2012Metric_Pad1.20x1.40mm_HandSolder, symbol Device:R_Small
- added C59, C60: 10u, Capacitor_SMD:C_0805_2012Metric_Pad1.18x1.45mm_HandSolder, symbol Device:C_Small
- added R47, R49: 4.7k, Resistor_SMD:R_0805_2012Metric_Pad1.20x1.40mm_HandSolder, symbol Device:R
Connections:
- net +3V3: now also C60.1, R47.2, R49.1
- net 3V3D: now also C59.2
- net GND: now also C60.2
- net GNDD: now also C59.1
- net SCL: now also R49.2
- net SDA: now also R47.1
