File: hardware/kinetic-pcb/sheets/led-mos.kicad_sch (KiCad schematic)
At the start: 3 parts, among them Q10 DMN2053UQ-13

Commit message: fixes pre-prod
Parts:
- Q10: footprint Package_TO_SOT_SMD:TSOT-23_HandSoldering -> Project:SOT-23_Handsoldering-DMN2053UQ
Changed lines of the file:
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@@
 			)
 		)
-		(property "Footprint" "Package_TO_SOT_SMD:TSOT-23_HandSoldering"
+		(property "Footprint" "Project:SOT-23_Handsoldering-DMN2053UQ"
 			(at 85.09 92.71 0)
 			(effects
