File: hardware/kinetic-pcb/sheets/pump.kicad_sch (KiCad schematic)
At the start: 7 parts, among them J15 MicroFit2x1, Q2 DMN2053UQ-13

Commit message: fixes pre-prod
Parts:
- Q2: footprint Package_TO_SOT_SMD:TSOT-23_HandSoldering -> Project:SOT-23_Handsoldering-DMN2053UQ
Changed lines of the file:
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@@
 			)
 		)
-		(property "Footprint" "Package_TO_SOT_SMD:TSOT-23_HandSoldering"
+		(property "Footprint" "Project:SOT-23_Handsoldering-DMN2053UQ"
 			(at 109.22 96.52 0)
 			(effects
